File: RP2040-Test.kicad_pcb (KiCad board)
At the start: 2 copper layers, 18.3 x 41.1 mm, 39 parts, among them J1 USB_B_Micro, J2 Conn_01x20, J3 Conn_01x20, J4 Conn_01x03, U1 MIC5205-3.3YM5, U2 RP2040, U3 W25Q32JVSS, Y1 Crystal_GND24_Small

Commit message: Fixed UL licensing with JLCPCB
Parts:
- removed the G*** at (101.4, 68.4)
Routing:
- net /QSPI_CS: track 19.7 -> 19.1 mm
- net GND: vias 19 -> 18
Other:
- board text added: "94V-0 E479892 JLC-2"
